File: r5.kicad_pcb (KiCad board)
At the start: 2 copper layers, 94.4 x 92.2 mm, 73 parts, among them J1 Conn_01x04, U1 LMZ22005, U10 74368PW, U100 Pico, U2 74LS365, U20 DRV8871DDA, U3 GY-BNO08X, U30 DRV8871DDA, U4 PI22, U40 DRV8871DDA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

Commit message: wip
Parts:
- added R15: 100k, Resistor_SMD:R_0805_2012Metric_Pad1.20x1.40mm_HandSolder, F.Cu at (83.0, 115.2)
- added R16: 100k, Resistor_SMD:R_0805_2012Metric_Pad1.20x1.40mm_HandSolder, F.Cu at (83.0, 118.2)
- added R17: 100k, Resistor_SMD:R_0805_2012Metric_Pad1.20x1.40mm_HandSolder, F.Cu at (83.0, 121.1)
- added SW1: SW_SPDT, _r5:SW_Slide_1P2T_CK_OS102011MS2Q, F.Cu at (95.4, 144.0)
- added SW2: SW_SPDT, _r5:SW_Slide_1P2T_CK_OS102011MS2Q, F.Cu at (93.2, 56.2)
- added SW3: SW_SPDT, _r5:SW_Slide_1P2T_CK_OS102011MS2Q, F.Cu at (93.0, 61.0)
- added SW4: SW_SPDT, _r5:SW_Slide_1P2T_CK_OS102011MS2Q, F.Cu at (92.9, 66.0)
- moved J1 26.7 mm to (73.0, 55.6), turned to -90 degrees
- moved X81 16.2 mm to (60.9, 69.1)
- moved U5 15.0 mm to (70.1, 59.0), turned to -90 degrees
- moved C4 14.4 mm to (115.8, 112.6)
- moved R11 12.5 mm to (112.0, 114.2)
- moved U80 9.08 mm to (83.8, 64.8)
- moved R20 6.86 mm to (126.2, 122.6)
- moved C81 5.97 mm to (85.4, 58.4)
- moved R40 5.15 mm to (126.6, 107.0)
- moved C70 5.09 mm to (131.0, 85.6)
- moved C30 5.03 mm to (131.0, 114.8)
- moved R30 4.88 mm to (126.0, 114.8)
- moved C50 4.80 mm to (131.0, 99.8)
- moved H2 4.40 mm to (74.6, 65.2)
- moved R60 4.31 mm to (126.4, 92.8)
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Connections:
- R10 pad 2: MENABLE -> Net-(SW2-C)
- R11 pad 1: +BATT -> Net-(SW1-B)
- U10 pad 1: MENABLE -> Net-(SW2-C)
- U10 pad 15: MENABLE -> Net-(SW2-C)
- U2 pad 1: MENABLE -> Net-(SW2-C)
- U2 pad 15: MENABLE -> Net-(SW2-C)
- U4 pad 11: unconnected-(U4-GPIO17-Pad11) -> INWIFI
- U80 pad 23: unconnected-(U80-~{OE}-Pad23) -> Net-(SW4-B)
Routing:
- net GND: track 263.5 -> 11.7 mm, vias 64 -> 16
- net +BATT: track 97.4 -> 2.40 mm, vias 6 -> 0
- net Net-(U20-OUT2): track 14.0 -> 0.00 mm
- net Net-(U60-OUT1): track 13.5 -> 0.00 mm
- net Net-(U40-OUT1): track 13.5 -> 0.00 mm
- net Net-(U40-OUT2): track 13.0 -> 0.00 mm
- net Net-(U30-OUT2): track 12.9 -> 0.00 mm
- net Net-(U30-OUT1): track 12.9 -> 0.00 mm
- net Net-(U60-OUT2): track 12.8 -> 0.00 mm
- net Net-(U50-OUT2): track 12.6 -> 0.00 mm
- net Net-(U50-OUT1): track 12.4 -> 0.00 mm
- net Net-(U70-OUT2): track 12.4 -> 0.00 mm
- net Net-(U70-OUT1): track 12.3 -> 0.00 mm
- net Net-(U20-OUT1): track 10.3 -> 0.00 mm
- net Net-(U70-ILIM): track 2.27 -> 0.00 mm
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