File: r5.kicad_sch (KiCad schematic)
At the start: 81 parts, among them SW10 SW_SPDT, SW60 SW_SPDT, SW70 SW_SPDT, SW80 SW_SPDT, U10 LMZ22005, U20 DRV8871DDA, U21 DRV8871DDA, U22 DRV8871DDA, U23 DRV8871DDA, U24 DRV8871DDA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

Commit message: routing done
Parts:
- R10: value 102k -> 22k; LCSC Part # C40372 -> C17560
- R11: value 13k7 -> 3k; LCSC Part # C17448 -> C17661
- U10: LCSC Part # (none) -> C2865843; now in the parts list
- renumbered SW10 to S10, SW60 to S60, SW70 to S70, SW80 to S80
Connections:
- net GND: no longer X10.1 (Pin_1), X11.1 (Pin_1), X11.2 (Pin_2)
- net GNDPWR: now also X10.1 (Pin_1), X11.1 (Pin_1), X11.2 (Pin_2)
Other:
- note added: "10.66V under voltage cutoff (3S LiPo) Vul = (R10/R11+1)*1.279"
- note added: "Output voltage 4.98V VO = 0.8V*(1 + R13/(R14+R15))"
- note removed: "10.8V under voltage cutoff (3S LiPo)"
Changed lines of the file:
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@@
     (effects (font (size 1.27 1.27)) (justify left bottom))
   )
-  (text "10.8V under voltage cutoff (3S LiPo)" (at 43.18 134.62 0)
+  (text "Output voltage 4.98V\nVO = 0.8V*(1 + R13/(R14+R15)) "
+    (at 81.28 138.43 0)
+    (effects (font (size 1.27 1.27)) (justify left bottom))
+  )
+  (text "10.66V under voltage cutoff (3S LiPo)\nVul = (R10/R11+1)*1.279"
+    (at 40.64 138.43 0)
     (effects (font (size 1.27 1.27)) (justify left bottom))
   )
@@
   )
   (symbol (lib_id "_r5:LMZ22005") (at 68.58 104.14 0) (unit 1)
-    (in_bom no) (on_board yes) (dnp no)
+    (in_bom yes) (on_board yes) (dnp no)
     (property "Reference" "U10" (at 68.58 92.329 0)
       (effects (font (size 1.27 1.27)))
@@
       (effects (font (size 1.27 1.27)) hide)
     )
+    (property "LCSC Part #" "C2865843" (at 68.58 104.14 0)
+      (effects (font (size 1.27 1.27)) hide)
+    )
     (pin "1")
     (pin "5")
@@
     )
   )
-  (symbol (lib_id "power:GND") (at 46.99 64.77 0) (unit 1)
-    (in_bom yes) (on_board yes) (dnp no)
-    (property "Reference" "#PWR0205" (at 46.99 71.12 0)
-      (effects (font (size 1.27 1.27)) hide)
-    )
-    (property "Value" "GND" (at 47.117 69.1642 0)
-      (effects (font (size 1.27 1.27)))
-    )
-    (property "Footprint" "" (at 46.99 64.77 0)
-      (effects (font (size 1.27 1.27)) hide)
-    )
-    (property "Datasheet" "" (at 46.99 64.77 0)
-      (effects (font (size 1.27 1.27)) hide)
-    )
-    (pin "1")
-    (instances
-      (project "r5"
-        (path "/7141c11d-0c81-438d-ad8c-6c0ffa292856"
-          (reference "#PWR0205") (unit 1)
-        )
-      )
-    )
-  )
   (symbol (lib_id "power:+BATT") (at 46.99 45.72 0) (unit 1)
     (in_bom yes) (on_board yes) (dnp no)
@@
     )
   )
-  (symbol (lib_id "power:GND") (at 87.63 64.77 0) (unit 1)
-    (in_bom yes) (on_board yes) (dnp no)
-    (property "Reference" "#PWR0214" (at 87.63 71.12 0)
-      (effects (font (size 1.27 1.27)) hide)
-    )
-    (property "Value" "GND" (at 87.757 69.1642 0)
-      (effects (font (size 1.27 1.27)))
-    )
-    (property "Footprint" "" (at 87.63 64.77 0)
-      (effects (font (size 1.27 1.27)) hide)
-    )
-    (property "Datasheet" "" (at 87.63 64.77 0)
-      (effects (font (size 1.27 1.27)) hide)
-    )
-    (pin "1")
-    (instances
-      (project "r5"
-        (path "/7141c11d-0c81-438d-ad8c-6c0ffa292856"
-          (reference "#PWR0214") (unit 1)
-        )
-      )
-    )
-  )
   (symbol (lib_id "Device:R") (at 62.23 49.53 0) (unit 1)
     (in_bom yes) (on_board yes) (dnp no)
@@
   (symbol (lib_id "Switch:SW_SPDT") (at 364.49 82.55 0) (unit 1)
     (in_bom no) (on_board yes) (dnp no) (fields_autoplaced)
-    (property "Reference" "SW70" (at 364.49 73.66 0)
+    (property "Reference" "S70" (at 364.49 73.66 0)
       (effects (font (size 1.27 1.27)))
     )
@@
       (project "r5"
         (path "/7141c11d-0c81-438d-ad8c-6c0ffa292856"
-          (reference "SW70") (unit 1)
+          (reference "S70") (unit 1)
         )
       )
@@
     )
   )
+  (symbol (lib_id "power:GNDPWR") (at 87.63 64.77 0) (unit 1)
+    (in_bom yes) (on_board yes) (dnp no)
+    (property "Reference" "#PWR051" (at 87.63 69.85 0)
+      (effects (font (size 1.27 1.27)) hide)
+    )
+    (property "Value" "GNDPWR" (at 87.7316 68.6816 0)
+      (effects (font (size 1.27 1.27)))
+    )
+    (property "Footprint" "" (at 87.63 66.04 0)
+      (effects (font (size 1.27 1.27)) hide)
+    )
+    (property "Datasheet" "" (at 87.63 66.04 0)
+      (effects (font (size 1.27 1.27)) hide)
+    )
+    (pin "1")
+    (instances
+      (project "r5"
+        (path "/7141c11d-0c81-438d-ad8c-6c0ffa292856"
+          (reference "#PWR051") (unit 1)
+        )
+      )
+    )
+  )
   (symbol (lib_id "power:GND") (at 199.39 252.73 0) (unit 1)
     (in_bom yes) (on_board yes) (dnp no) (fields_autoplaced)
@@
       (effects (font (size 1.27 1.27)) (justify left))
     )
-    (property "Value" "13k7" (at 42.418 130.683 0)
+    (property "Value" "3k" (at 42.418 130.683 0)
       (effects (font (size 1.27 1.27)) (justify left))
     )
@@
       (effects (font (size 1.27 1.27)) hide)
     )
-    (property "LCSC Part #" "C17448" (at 40.64 129.54 0)
+    (property "LCSC Part #" "C17661" (at 40.64 129.54 0)
       (effects (font (size 1.27 1.27)) hide)
     )
@@
   (symbol (lib_id "Switch:SW_SPDT") (at 306.07 158.75 0) (unit 1)
     (in_bom no) (on_board yes) (dnp no) (fields_autoplaced)
-    (property "Reference" "SW60" (at 306.07 149.86 0)
+    (property "Reference" "S60" (at 306.07 149.86 0)
       (effects (font (size 1.27 1.27)))
     )
@@
       (project "r5"
         (path "/7141c11d-0c81-438d-ad8c-6c0ffa292856"
-          (reference "SW60") (unit 1)
+          (reference "S60") (unit 1)
         )
       )
@@
   (symbol (lib_id "Switch:SW_SPDT") (at 194.31 255.27 0) (unit 1)
     (in_bom no) (on_board yes) (dnp no) (fields_autoplaced)
-    (property "Reference" "SW80" (at 194.31 246.38 0)
+    (property "Reference" "S80" (at 194.31 246.38 0)
       (effects (font (size 1.27 1.27)))
     )
@@
       (project "r5"
         (path "/7141c11d-0c81-438d-ad8c-6c0ffa292856"
-          (reference "SW80") (unit 1)
+          (reference "S80") (unit 1)
         )
       )
@@
   (symbol (lib_id "Switch:SW_SPDT") (at 40.64 110.49 0) (unit 1)
     (in_bom no) (on_board yes) (dnp no) (fields_autoplaced)
-    (property "Reference" "SW10" (at 40.64 101.6 0)
+    (property "Reference" "S10" (at 40.64 101.6 0)
       (effects (font (size 1.27 1.27)))
     )
@@
       (project "r5"
         (path "/7141c11d-0c81-438d-ad8c-6c0ffa292856"
-          (reference "SW10") (unit 1)
+          (reference "S10") (unit 1)
         )
       )
@@
     )
   )
+  (symbol (lib_id "power:GNDPWR") (at 46.99 64.77 0) (unit 1)
+    (in_bom yes) (on_board yes) (dnp no)
+    (property "Reference" "#PWR052" (at 46.99 69.85 0)
+      (effects (font (size 1.27 1.27)) hide)
+    )
+    (property "Value" "GNDPWR" (at 47.0916 68.6816 0)
+      (effects (font (size 1.27 1.27)))
+    )
+    (property "Footprint" "" (at 46.99 66.04 0)
+      (effects (font (size 1.27 1.27)) hide)
+    )
+    (property "Datasheet" "" (at 46.99 66.04 0)
+      (effects (font (size 1.27 1.27)) hide)
+    )
+    (pin "1")
+    (instances
+      (project "r5"
+        (path "/7141c11d-0c81-438d-ad8c-6c0ffa292856"
+          (reference "#PWR052") (unit 1)
+        )
+      )
+    )
+  )
   (symbol (lib_id "74xx:74LS540") (at 397.51 107.95 0) (unit 1)
     (in_bom yes) (on_board yes) (dnp no) (fields_autoplaced)
@@
       (effects (font (size 1.27 1.27)) (justify left))
     )
-    (property "Value" "102k" (at 42.418 123.063 0)
+    (property "Value" "22k" (at 42.418 123.063 0)
       (effects (font (size 1.27 1.27)) (justify left))
     )
@@
       (effects (font (size 1.27 1.27)) hide)
     )
-    (property "LCSC Part #" "C40372" (at 40.64 121.92 0)
+    (property "LCSC Part #" "C17560" (at 40.64 121.92 0)
       (effects (font (size 1.27 1.27)) hide)
     )

Commit message: Silk cleanup
Parts:
- U10: now left out of the parts list
Changed lines of the file:
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@@
   )
   (symbol (lib_id "_r5:LMZ22005") (at 68.58 104.14 0) (unit 1)
-    (in_bom yes) (on_board yes) (dnp no)
+    (in_bom no) (on_board yes) (dnp no)
     (property "Reference" "U10" (at 68.58 92.329 0)
       (effects (font (size 1.27 1.27)))

Commit message: board done
Parts:
- U20, U21, U22, U23, U24, U25: footprint Package_SO:Texas_HTSOP-8-1EP_3.9x4.9mm_P1.27mm_EP2.95x4.9mm_Mask2.4x3.1mm_ThermalVias -> _r5:Texas_HTSOP-8-1EP_3.9x4.9mm_P1.27mm_EP2.95x4.9mm_Mask2.4x3.1mm_ThermalVias
Changed lines of the file:
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@@
       (effects (font (size 1.27 1.27)))
     )
-    (property "Footprint" "Package_SO:Texas_HTSOP-8-1EP_3.9x4.9mm_P1.27mm_EP2.95x4.9mm_Mask2.4x3.1mm_ThermalVias" (at 163.83 66.04 0)
+    (property "Footprint" "_r5:Texas_HTSOP-8-1EP_3.9x4.9mm_P1.27mm_EP2.95x4.9mm_Mask2.4x3.1mm_ThermalVias" (at 163.83 66.04 0)
       (effects (font (size 1.27 1.27)) hide)
     )
@@
       (effects (font (size 1.27 1.27)))
     )
-    (property "Footprint" "Package_SO:Texas_HTSOP-8-1EP_3.9x4.9mm_P1.27mm_EP2.95x4.9mm_Mask2.4x3.1mm_ThermalVias" (at 163.83 101.6 0)
+    (property "Footprint" "_r5:Texas_HTSOP-8-1EP_3.9x4.9mm_P1.27mm_EP2.95x4.9mm_Mask2.4x3.1mm_ThermalVias" (at 163.83 101.6 0)
       (effects (font (size 1.27 1.27)) hide)
     )
@@
       (effects (font (size 1.27 1.27)))
     )
-    (property "Footprint" "Package_SO:Texas_HTSOP-8-1EP_3.9x4.9mm_P1.27mm_EP2.95x4.9mm_Mask2.4x3.1mm_ThermalVias" (at 219.71 29.21 0)
+    (property "Footprint" "_r5:Texas_HTSOP-8-1EP_3.9x4.9mm_P1.27mm_EP2.95x4.9mm_Mask2.4x3.1mm_ThermalVias" (at 219.71 29.21 0)
       (effects (font (size 1.27 1.27)) hide)
     )
@@
       (effects (font (size 1.27 1.27)))
     )
-    (property "Footprint" "Package_SO:Texas_HTSOP-8-1EP_3.9x4.9mm_P1.27mm_EP2.95x4.9mm_Mask2.4x3.1mm_ThermalVias" (at 219.71 64.77 0)
+    (property "Footprint" "_r5:Texas_HTSOP-8-1EP_3.9x4.9mm_P1.27mm_EP2.95x4.9mm_Mask2.4x3.1mm_ThermalVias" (at 219.71 64.77 0)
       (effects (font (size 1.27 1.27)) hide)
     )
@@
       (effects (font (size 1.27 1.27)))
     )
-    (property "Footprint" "Package_SO:Texas_HTSOP-8-1EP_3.9x4.9mm_P1.27mm_EP2.95x4.9mm_Mask2.4x3.1mm_ThermalVias" (at 219.71 101.6 0)
+    (property "Footprint" "_r5:Texas_HTSOP-8-1EP_3.9x4.9mm_P1.27mm_EP2.95x4.9mm_Mask2.4x3.1mm_ThermalVias" (at 219.71 101.6 0)
       (effects (font (size 1.27 1.27)) hide)
     )
@@
       (effects (font (size 1.27 1.27)))
     )
-    (property "Footprint" "Package_SO:Texas_HTSOP-8-1EP_3.9x4.9mm_P1.27mm_EP2.95x4.9mm_Mask2.4x3.1mm_ThermalVias" (at 163.83 30.48 0)
-      (effects (font (size 1.27 1.27)) hide)
-    )
+    (property "Footprint" "_r5:Texas_HTSOP-8-1EP_3.9x4.9mm_P1.27mm_EP2.95x4.9mm_Mask2.4x3.1mm_ThermalVias" (at 163.83 30.48 0)
+      (effects (font (size 1.27 1.27)) hide)
+    )
